Commit message: Established connection between JSP GUI and Gazebo

File: Project2/project2/models/ur5_rg2/model_minimal.urdf (robot description, URDF)
Before this commit: robot ur5_rg2, 12 links, 11 joints
Links:
- link base_link: geometry visual mesh filename=package://project2/models/ur5_rg2/meshes/visual/ur5/base.dae scale=1 1 1
- link forearm_link: geometry visual mesh filename=package://project2/models/ur5_rg2/meshes/visual/ur5/forearm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 scale=1 1 1
- link rg2_hand: geometry visual mesh filename=package://project2/models/ur5_rg2/meshes/visual/rg2/hand.dae scale=1 1 1
- link rg2_leftfinger: geometry visual mesh filename=package://project2/models/ur5_rg2/meshes/visual/rg2/finger.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 scale=1 1 1
- link rg2_rightfinger: geometry visual mesh filename=package://project2/models/ur5_rg2/meshes/visual/rg2/finger.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 scale=1 1 1
- link shoulder_link: geometry visual mesh filename=package://project2/models/ur5_rg2/meshes/visual/ur5/shoulde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 scale=1 1 1
- link upper_arm_link: geometry visual mesh filename=package://project2/models/ur5_rg2/meshes/visual/ur5/upperar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 scale=1 1 1
- link wrist_1_link: geometry visual mesh filename=package://project2/models/ur5_rg2/meshes/visual/ur5/wrist1.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 scale=1 1 1
- link wrist_2_link: geometry visual mesh filename=package://project2/models/ur5_rg2/meshes/visual/ur5/wrist2.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 scale=1 1 1
- link wrist_3_link: geometry visual mesh filename=package://project2/models/ur5_rg2/meshes/visual/ur5/wrist3.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 scale=1 1 1
Joints:
- joint rg2_finger_joint1: axis (none) -> 0.0 0.0 1.0
- joint rg2_finger_joint2: axis (none) -> 0.0 0.0 -1.0
